File: rover-mppt-pcb/rover-mppt-pcb.kicad_sch (KiCad schematic)
At the start: 26 parts, among them J1 OC, Q1 SiR880BDP, Q2 SiR880BDP, U1 BQ25820RRVR

Commit message: Created thermal DAQ
Parts:
- added J2: Conn_01x10, Connector_Molex:Molex_PicoBlade_53047-1010_1x10_P1.25mm_Vertical, symbol Connector_Generic:Conn_01x10
- R1, R4: footprint (none) -> Resistor_SMD:R_2512_6332Metric
- R2, R3, R5, R_{CHG}1, R_{FS}1, R_{LIM}1, R_{SNS}1: footprint (none) -> Resistor_SMD:R_1206_3216Metric
- R_{SNS}2: footprint (none) -> Resistor_SMD:R_2010_5025Metric
- U1: value BQ25820RRVR -> BQ25822RRVR
Connections:
- net GND: now also J2.10 (Pin_10); no longer R3.2
- net I2C_SCL: now also J2.7 (Pin_7)
- net I2C_SDA: now also J2.6 (Pin_6)
- net VCC: now also J2.9 (Pin_9)
- net ~{CE}: now also J2.8 (Pin_8)
- net ~{INT}: now also J2.5 (Pin_5)
- net GNDREF: now reaches U1.11 (FBG)
- net GNDREF: now also R3.2
- no-connect marks 7 -> 6
Other:
- moved on the sheet: C7, D1, R4, R5, U1
