File: temp-adc/temp-adc.kicad_sch (KiCad schematic)
At the start: 22 parts, among them J1 Conn_01x06, U1 MCP3204

Commit message: New PCB using MCP3428-SL
Parts:
- removed C1, C2, C3, C4: 5600p, Capacitor_SMD:C_1206_3216Metric_Pad1.33x1.80mm_HandSolder, symbol Device:C
- removed U1: MCP3204, Package_SO:SOIC-14_3.9x8.7mm_P1.27mm, symbol Analog_ADC:MCP3204
- added JP1, JP2: SolderJumper_3_Open, Jumper:SolderJumper-3_P2.0mm_Open_TrianglePad1.0x1.5mm, symbol Jumper:SolderJumper_3_Open
- added U2: MCP3428x-xSL, Package_SO:SOIC-14_3.9x8.7mm_P1.27mm, symbol Analog_ADC:MCP3428x-xSL
- H1, H2, H3, H4: footprint MountingHole:MountingHole_M2.5_thinoutline -> footprints:MountingHole_M2_dia0.1in
Connections:
- net GND: now also JP1.3 (B), JP2.3 (B), U2.12 (CH3-), U2.14 (CH4-), U2.2 (CH1-), U2.4 (CH2-), U2.5 (V_{SS})
- net IN0: now also U2.13 (CH4+)
- net IN1: now also U2.11 (CH3+)
- net IN2: now also U2.3 (CH2+)
- net IN3: now also U2.1 (CH1+)
- net VCC: now also JP1.1 (A), JP2.1 (A), U2.6 (V_{DD})
- net MISO renamed SDA
- net SDA: now also U2.7 (SDA)
- net MOSI renamed A1
- net A1: now also JP2.2 (C), U2.10 (Adr1)
- net SCK renamed SCL
- net SCL: now also U2.8 (SCL)
- net ~{CS} renamed A0
- net A0: now also JP1.2 (C), U2.9 (Adr0)
Other:
- moved on the sheet: J1
